Commit message: version 0.2.1 simplify the ludan mesh, now can load the model really quick

File: src/ludan_moveit_config/config/gazebo_ludan_v0.urdf (robot description, URDF)
Before this commit: robot ludan_v0, 31 links, 30 joints
Links:
- link Body: geometry collision mesh filename=package://ludan_v0/simplified_meshes/Body.STL; visual mesh filename=package://ludan_v0/simplified_meshes/Body.STL
- link LeftAnklePitch: geometry collision mesh filename=package://ludan_v0/simplified_meshes/LeftAnklePitch.STL; visual mesh filename=package://ludan_v0/simplified_meshes/LeftAnklePitch.STL
- link LeftAnkleRoll: geometry collision mesh filename=package://ludan_v0/simplified_meshes/LeftAnkleRoll.STL; visual mesh filename=package://ludan_v0/simplified_meshes/LeftAnkleRoll.STL
- link LeftElbowPitch: geometry collision mesh filename=package://ludan_v0/simplified_meshes/LeftElbowPitch.STL; visual mesh filename=package://ludan_v0/simplified_meshes/LeftElbowPitch.STL
- link LeftElbowYaw: geometry collision mesh filename=package://ludan_v0/simplified_meshes/LeftElbowYaw.STL; visual mesh filename=package://ludan_v0/simplified_meshes/LeftElbowYaw.STL
- link LeftHipPitch: geometry collision mesh filename=package://ludan_v0/simplified_meshes/LeftHipPitch.STL; visual mesh filename=package://ludan_v0/simplified_meshes/LeftHipPitch.STL
- link LeftHipRoll: geometry collision mesh filename=package://ludan_v0/simplified_meshes/LeftHipRoll.STL; visual mesh filename=package://ludan_v0/simplified_meshes/LeftHipRoll.STL
- link LeftHipYaw: geometry collision mesh filename=package://ludan_v0/simplified_meshes/LeftHipYaw.STL; visual mesh filename=package://ludan_v0/simplified_meshes/LeftHipYaw.STL
- link LeftKnee: geometry collision mesh filename=package://ludan_v0/simplified_meshes/LeftKnee.STL; visual mesh filename=package://ludan_v0/simplified_meshes/LeftKnee.STL
- link LeftShoulderPitch: geometry collision mesh filename=package://ludan_v0/simplified_meshes/LeftShoulderPitch.STL; visual mesh filename=package://ludan_v0/simplified_meshes/LeftShoulderPitch.STL
- link LeftShoulderRoll: geometry collision mesh filename=package://ludan_v0/simplified_meshes/LeftShoulderRoll.STL; visual mesh filename=package://ludan_v0/simplified_meshes/LeftShoulderRoll.STL
- link LeftShoulderYaw: geometry collision mesh filename=package://ludan_v0/simplified_meshes/LeftShoulderYaw.STL; visual mesh filename=package://ludan_v0/simplified_meshes/LeftShoulderYaw.STL
- link LeftWristPitch: geometry collision mesh filename=package://ludan_v0/simplified_meshes/LeftWristPitch.STL; visual mesh filename=package://ludan_v0/simplified_meshes/LeftWristPitch.STL
- link LeftWristRoll: geometry collision mesh filename=package://ludan_v0/simplified_meshes/LeftWristRoll.STL; visual mesh filename=package://ludan_v0/simplified_meshes/LeftWristRoll.STL
- link NeckPitch: geometry collision mesh filename=package://ludan_v0/simplified_meshes/NeckPitch.STL; visual mesh filename=package://ludan_v0/simplified_meshes/NeckPitch.STL
- link NeckRoll: geometry collision mesh filename=package://ludan_v0/simplified_meshes/NeckRoll.STL; visual mesh filename=package://ludan_v0/simplified_meshes/NeckRoll.STL
- link NeckYaw: geometry collision mesh filename=package://ludan_v0/simplified_meshes/NeckYaw.STL; visual mesh filename=package://ludan_v0/simplified_meshes/NeckYaw.STL
- link RightAnklePitch: geometry collision mesh filename=package://ludan_v0/simplified_meshes/RightAnklePitch.STL; visual mesh filename=package://ludan_v0/simplified_meshes/RightAnklePitch.STL
- link RightAnkleRoll: geometry collision mesh filename=package://ludan_v0/simplified_meshes/RightAnkleRoll.STL; visual mesh filename=package://ludan_v0/simplified_meshes/RightAnkleRoll.STL
- link RightElbowPitch: geometry collision mesh filename=package://ludan_v0/simplified_meshes/RightElbowPitch.STL; visual mesh filename=package://ludan_v0/simplified_meshes/RightElbowPitch.STL
- link RightElbowYaw: geometry collision mesh filename=package://ludan_v0/simplified_meshes/RightElbowYaw.STL; visual mesh filename=package://ludan_v0/simplified_meshes/RightElbowYaw.STL
- link RightHipPitch: geometry collision mesh filename=package://ludan_v0/simplified_meshes/RightHipPitch.STL; visual mesh filename=package://ludan_v0/simplified_meshes/RightHipPitch.STL
- link RightHipRoll: geometry collision mesh filename=package://ludan_v0/simplified_meshes/RightHipRoll.STL; visual mesh filename=package://ludan_v0/simplified_meshes/RightHipRoll.STL
- link RightHipYaw: geometry collision mesh filename=package://ludan_v0/simplified_meshes/RightHipYaw.STL; visual mesh filename=package://ludan_v0/simplified_meshes/RightHipYaw.STL
- link RightKnee: geometry collision mesh filename=package://ludan_v0/simplified_meshes/RightKnee.STL; visual mesh filename=package://ludan_v0/simplified_meshes/RightKnee.STL
- link RightShoulderPitch: geometry collision mesh filename=package://ludan_v0/simplified_meshes/RightShoulderPitch.STL; visual mesh filename=package://ludan_v0/simplified_meshes/RightShoulderPitch.STL
- link RightShoulderRoll: geometry collision mesh filename=package://ludan_v0/simplified_meshes/RightShoulderRoll.STL; visual mesh filename=package://ludan_v0/simplified_meshes/RightShoulderRoll.STL
- link RightShoulderYaw: geometry collision mesh filename=package://ludan_v0/simplified_meshes/RightShoulderYaw.STL; visual mesh filename=package://ludan_v0/simplified_meshes/RightShoulderYaw.STL
- link RightWristPitch: geometry collision mesh filename=package://ludan_v0/simplified_meshes/RightWristPitch.STL; visual mesh filename=package://ludan_v0/simplified_meshes/RightWristPitch.STL
- link RightWristRoll: geometry collision mesh filename=package://ludan_v0/simplified_meshes/RightWristRoll.STL; visual mesh filename=package://ludan_v0/simplified_meshes/RightWristRoll.STL
- link WaistYaw: geometry collision mesh filename=package://ludan_v0/simplified_meshes/WaistYaw.STL; visual mesh filename=package://ludan_v0/simplified_meshes/WaistYaw.STL
